Commit message: planning adapter works, need some clean up

File: omnid/urdf/delta_robot.urdf (robot description, URDF)
Before this commit: robot delta-robot-RUU, 26 links, 25 joints
Links:
- added link extra_knee_link_1
- added link extra_knee_link_2
- added link extra_knee_link_3
- added link mimic_knee_link_1
- added link mimic_knee_link_2
- added link mimic_knee_link_3
- added link mimic_lower_leg_1
- added link mimic_lower_leg_2
- added link mimic_lower_leg_3
Joints:
- added joint extra_knee_lower_leg_1: type fixed, parent extra_knee_link_1, child mimic_lower_leg_1, origin xyz=-0.2 0 0 rpy=0 0 0
- added joint extra_knee_lower_leg_2: type fixed, parent extra_knee_link_2, child mimic_lower_leg_2, origin xyz=-0.2 0 0 rpy=0 0 0
- added joint extra_knee_lower_leg_3: type fixed, parent extra_knee_link_3, child mimic_lower_leg_3, origin xyz=-0.2 0 0 rpy=0 0 0
- added joint mimic_beta_1: type continuous, parent mimic_knee_link_1, child extra_knee_link_1, origin xyz=1e-5 1e-5 1e-5 rpy=0 0 0, axis 0 -1 0, mimic joint=beta_1 multiplier=-1 offset=0
- added joint mimic_beta_2: type continuous, parent mimic_knee_link_2, child extra_knee_link_2, origin xyz=1e-5 1e-5 1e-5 rpy=0 0 0, axis 0 -1 0, mimic joint=beta_2 multiplier=-1 offset=0
- added joint mimic_beta_3: type continuous, parent mimic_knee_link_3, child extra_knee_link_3, origin xyz=1e-5 1e-5 1e-5 rpy=0 0 0, axis 0 -1 0, mimic joint=beta_3 multiplier=-1 offset=0
- added joint mimic_gamma_1: type continuous, parent upper_leg_1, child mimic_knee_link_1, axis 0 0 -1, mimic joint=gamma_1 multiplier=-1 offset=0
- added joint mimic_gamma_2: type continuous, parent upper_leg_2, child mimic_knee_link_2, axis 0 0 -1, mimic joint=gamma_2 multiplier=-1 offset=0
- added joint mimic_gamma_3: type continuous, parent upper_leg_3, child mimic_knee_link_3, axis 0 0 -1, mimic joint=gamma_3 multiplier=-1 offset=0
- joint lower_leg_attach_joint_2: origin xyz=-0.08999999999999996 0.15588457268119896 0 rpy=0 0 2.0943951023931953 -> xyz=-0.09 0.155884572681 0 rpy=0 0 2.09439510239
- joint lower_leg_attach_joint_3: origin xyz=-0.09000000000000008 -0.1558845726811989 0 rpy=0 0 4.1887902047863905 -> xyz=-0.09 -0.155884572681 0 rpy=0 0 4.18879020479
- joint mimic_theta_1: limit lower=-1.5707963267948966 upper=1.5707963267948966 effort=100 velocity=100 -> lower=-1.57079632679 upper=1.57079632679 effort=100 velocity=100; parent lower_leg_1 -> mimic_lower_leg_1
- joint mimic_theta_2: limit lower=-1.5707963267948966 upper=1.5707963267948966 effort=100 velocity=100 -> lower=-1.57079632679 upper=1.57079632679 effort=100 velocity=100; parent lower_leg_2 -> mimic_lower_leg_2
- joint mimic_theta_3: limit lower=-1.5707963267948966 upper=1.5707963267948966 effort=100 velocity=100 -> lower=-1.57079632679 upper=1.57079632679 effort=100 velocity=100; parent lower_leg_3 -> mimic_lower_leg_3
- joint mimic_theta_link_floating_world_2: origin xyz=-0.18 0 0 rpy=0 0 -2.0943951023931953 -> xyz=-0.18 0 0 rpy=0 0 -2.09439510239
- joint mimic_theta_link_floating_world_3: origin xyz=-0.18 0 0 rpy=0 0 -4.1887902047863905 -> xyz=-0.18 0 0 rpy=0 0 -4.18879020479
- joint phi_1: origin xyz=0 -0.09 0 rpy=0 0 1.5707963267948966 -> xyz=0 -0.09 0 rpy=0 0 1.57079632679
- joint phi_2: origin xyz=0 -0.09 0 rpy=0 0 1.5707963267948966 -> xyz=0 -0.09 0 rpy=0 0 1.57079632679
- joint phi_3: origin xyz=0 -0.09 0 rpy=0 0 1.5707963267948966 -> xyz=0 -0.09 0 rpy=0 0 1.57079632679
- joint theta_1: limit lower=-0.7853981633974483 upper=1.5707963267948966 effort=100 velocity=100 -> lower=-0.785398163397 upper=1.57079632679 effort=100 velocity=100
- joint theta_2: limit lower=-0.7853981633974483 upper=1.5707963267948966 effort=100 velocity=100 -> lower=-0.785398163397 upper=1.57079632679 effort=100 velocity=100
- joint theta_3: limit lower=-0.7853981633974483 upper=1.5707963267948966 effort=100 velocity=100 -> lower=-0.785398163397 upper=1.57079632679 effort=100 velocity=100
- joint z: limit lower=-0.046375 upper=0.5680000000000001 effort=100 velocity=100 -> lower=-0.046375 upper=0.568 effort=100 velocity=100

File: omnid/urdf/delta_robot_for_moveit.urdf.xacro (robot description, xacro)
@@ -223,5 +223,19 @@
         <dynamics damping="0.0" friction="0.0"/>
       </joint>
-      <!-- define the lower leg link -->
+    <!-- define the pre-spring link -->
+    <xacro:cylinder_link name="lower_leg_prespring_${id}"
+                         M="${M_prespring}"
+                         R="${R_prespring}"
+                         h="${h_prespring}"
+                         axis="x"
+                         mat="prespring_color" />
+    <joint name="phi_${id}" type="continuous">
+      <parent link="lower_leg_attach_link_${id}" />
+      <child link="lower_leg_prespring_${id}" />
+      <origin xyz="0 -${prespring_offset} 0" rpy="0 0 ${pi/2.0}" />
+      <axis xyz = "-1 0 0" rpy="0 0 0" />
+      <dynamics damping="0.0" friction="0.0"/>
+    </joint>
+    <!-- define the lower leg link -->
       <xacro:cylinder_link name="lower_leg_${id}"
                            M="${M_lower}"
@@ -240,37 +254,4 @@
         <dynamics damping="0.0" friction="0.0"/>
       </joint>
-      <!--      the chain for serialization -->
-    <joint name="mimic_theta_${id}" type="revolute">
-      <parent link="lower_leg_${id}" />
-      <child link="mimic_theta_link_${id}" />
-      <origin xyz="0 0 0" rpy="0 0 0" />
-      <axis xyz = "0 -1 0" rpy="0 0 0"/>
-      <limit lower="${-pi/2.0}" upper="${pi/2.0}" effort="100" velocity="100" />
-      <dynamics damping="0.0" friction="0.0"/>
-      <mimic joint="theta_${id}" multiplier="-1" offset="0"/>
-    </joint>
-    <link name="mimic_theta_link_${id}"/>
-    <joint name="mimic_theta_link_floating_world_${id}" type="fixed">
-      <parent link="mimic_theta_link_${id}" />
-      <child link="floating_world_${id}" />
-      <origin xyz="${-R_base} 0 0" rpy="0 0 ${-offset}" />
-      <dynamics damping="0.0" friction="0.0"/>
-    </joint>
-    <link name="floating_world_${id}"/>
-    <!--The chain for serialization ends here-->
-    <!-- define the pre-spring link -->
-    <xacro:cylinder_link name="lower_leg_prespring_${id}"
-                         M="${M_prespring}"
-                         R="${R_prespring}"
-                         h="${h_prespring}"
-                         axis="x"
-                         mat="prespring_color" />
-    <joint name="phi_${id}" type="continuous">
-      <parent link="lower_leg_attach_link_${id}" />
-      <child link="lower_leg_prespring_${id}" />
-      <origin xyz="0 -${prespring_offset} 0" rpy="0 0 ${pi/2.0}" />
-      <axis xyz = "-1 0 0" rpy="0 0 0" />
-      <dynamics damping="0.0" friction="0.0"/>
-    </joint>
       <!-- define a frame at the knee between the lower and upper legs -->
       <link name="knee_${id}" >
@@ -300,4 +281,46 @@
         <dynamics damping="0.0" friction="0.0"/>
       </joint>
+    <!--      the chain for serialization -->
+    <joint name="mimic_gamma_${id}" type="continuous">
+      <parent link="upper_leg_${id}" />
+      <child link="mimic_knee_link_${id}" />
+      <axis xyz="0 0 -1" rpy="0 0 0" />
+      <dynamics damping="0.0" friction="0.0"/>
+      <mimic joint="gamma_${id}" multiplier="-1" offset="0"/>
+    </joint>
+    <link name="mimic_knee_link_${id}"/>
+    <joint name="mimic_beta_${id}" type="continuous">
+      <parent link="mimic_knee_link_${id}" />
+      <child link="extra_knee_link_${id}" />
+      <origin xyz="0 0 0" rpy="0 0 0" />
+      <axis xyz="0 -1 0" rpy="0 0 0" />
+      <dynamics damping="0.0" friction="0.0"/>
+      <mimic joint="beta_${id}" multiplier="-1" offset="0"/>
+    </joint>
+    <link name="extra_knee_link_${id}"/>
+    <joint name="extra_knee_lower_leg_${id}" type="fixed">
+      <parent link="extra_knee_link_${id}" />
+      <child link="mimic_lower_leg_${id}" />
+      <origin xyz="${-L_lower} 0 0" rpy="0 0 0" />
+    </joint>
+    <link name="mimic_lower_leg_${id}"/>
+    <joint name="mimic_theta_${id}" type="revolute">
+      <parent link="mimic_lower_leg_${id}" />
+      <child link="mimic_theta_link_${id}" />
+      <origin xyz="0 0 0" rpy="0 0 0" />
+      <axis xyz = "0 -1 0" rpy="0 0 0"/>
+      <limit lower="${-pi/2.0}" upper="${pi/2.0}" effort="100" velocity="100" />
+      <dynamics damping="0.0" friction="0.0"/>
+      <mimic joint="theta_${id}" multiplier="-1" offset="0"/>
+    </joint>
+    <link name="mimic_theta_link_${id}"/>
+    <joint name="mimic_theta_link_floating_world_${id}" type="fixed">
+      <parent link="mimic_theta_link_${id}" />
+      <child link="floating_world_${id}" />
+      <origin xyz="${-R_base} 0 0" rpy="0 0 ${-offset}" />
+      <dynamics damping="0.0" friction="0.0"/>
+    </joint>
+    <link name="floating_world_${id}"/>
+    <!--The chain for serialization ends here-->
   </xacro:macro>
   <xacro:leg id="1" offset="0" head="True"/>

File: omnid/urdf/delta_robot_pybullet.urdf (robot description, URDF)
Before this commit: robot delta-robot-RUU, 20 links, 19 joints
Joints:
- joint lower_leg_attach_joint_2: origin xyz=-0.08999999999999996 0.15588457268119896 0 rpy=0 0 2.0943951023931953 -> xyz=-0.09 0.155884572681 0 rpy=0 0 2.09439510239
- joint lower_leg_attach_joint_3: origin xyz=-0.09000000000000008 -0.1558845726811989 0 rpy=0 0 4.1887902047863905 -> xyz=-0.09 -0.155884572681 0 rpy=0 0 4.18879020479
- joint phi_1: origin xyz=0 -0.09 0 rpy=0 0 1.5707963267948966 -> xyz=0 -0.09 0 rpy=0 0 1.57079632679
- joint phi_2: origin xyz=0 -0.09 0 rpy=0 0 1.5707963267948966 -> xyz=0 -0.09 0 rpy=0 0 1.57079632679
- joint phi_3: origin xyz=0 -0.09 0 rpy=0 0 1.5707963267948966 -> xyz=0 -0.09 0 rpy=0 0 1.57079632679
- joint theta_1: limit lower=-0.7853981633974483 upper=1.5707963267948966 effort=100 velocity=100 -> lower=-0.785398163397 upper=1.57079632679 effort=100 velocity=100
- joint theta_2: limit lower=-0.7853981633974483 upper=1.5707963267948966 effort=100 velocity=100 -> lower=-0.785398163397 upper=1.57079632679 effort=100 velocity=100
- joint theta_3: limit lower=-0.7853981633974483 upper=1.5707963267948966 effort=100 velocity=100 -> lower=-0.785398163397 upper=1.57079632679 effort=100 velocity=100
- joint z: limit lower=-0.046375 upper=0.5680000000000001 effort=100 velocity=100 -> lower=-0.046375 upper=0.568 effort=100 velocity=100

Commit message: multiple arms work in Pybullet, the current moveit package is not working this version

File: omnid/urdf/delta_robot.urdf (robot description, URDF)
Before this commit: robot delta-robot-RUU, 35 links, 34 joints
Joints:
- joint mimic_beta_1: origin xyz=1e-5 1e-5 1e-5 rpy=0 0 0 -> xyz=0 0 0 rpy=0 0 0
- joint mimic_beta_2: origin xyz=1e-5 1e-5 1e-5 rpy=0 0 0 -> xyz=0 0 0 rpy=0 0 0
- joint mimic_beta_3: origin xyz=1e-5 1e-5 1e-5 rpy=0 0 0 -> xyz=0 0 0 rpy=0 0 0

File: omnid/urdf/delta_robot_moveit.urdf.xacro (robot description, xacro)
@@ -111,5 +111,5 @@
       <xacro:cylinder_visual M="${M}" R="${R}" h="${h}" axis="${axis}" mat="${mat}" />
       <xacro:cylinder_inertia M="${M}" R="${R}" h="${h}" axis="${axis}" />
-      <xacro:cylinder_collision M="${M}" R="${R}" h="${h}" axis="{axis}"/>
+      <xacro:cylinder_collision M="${M}" R="${R}" h="${h}" axis="${axis}"/>
     </link>
   </xacro:macro>

File: omnid/urdf/delta_robot_pybullet.urdf.xacro (robot description, xacro)
@@ -64,5 +64,5 @@
       <!-- shift the origin to the center of the link from the end. how this is done depends on if
       the cylinder is x aligned or z aligned-->
-      <origin xyz="${0 if axis =='z' else h/2.0} 0 ${h/2.0 if axis=='z' else 0}" rpy="0 0 0" />
+<!--      <origin xyz="${0 if axis =='z' else h/2.0} 0 ${h/2.0 if axis=='z' else 0}" rpy="0 0 0" />-->
       <!-- formulas for inertia matrix components along radial and axial axes -->
       <xacro:property name="Iradial" value = "${M*h**2/12.0 + M*R**2/4.0}"/>
@@ -110,5 +110,5 @@
         <xacro:cylinder_visual M="${M}" R="${R}" h="${h}" axis="${axis}" mat="${mat}" />
         <xacro:cylinder_inertia M="${M}" R="${R}" h="${h}" axis="${axis}" />
-        <xacro:cylinder_collision M="${M}" R="${R}" h="${h}" axis="{axis}"/>
+        <xacro:cylinder_collision M="${M}" R="${R}" h="${h}" axis="${axis}"/>
       </link>
     </xacro:macro>
