Commit message: planner working with proper visualization

File: omnid/urdf/delta_robot_group_moveit.urdf.xacro (robot description, xacro)
@@ -80,4 +80,10 @@
   <xacro:property name="object_platform_base_y" value="${(robot_1_base_y + robot_2_base_y + robot_3_base_y)/3.0}"/>
   <xacro:property name="object_platform_base_z" value="${(robot_1_base_z + robot_2_base_z + robot_3_base_z)/3.0}"/>
+<!--TODO: organize your yaml params -->
+  <xacro:property name="yaml_file" value="$(find omnid)/params/params.yaml"/>
+  <xacro:property name="yaml_params" value="${load_yaml(yaml_file)}"/>
+  <xacro:property name="object_clearance" value="${yaml_params['object_clearance']}"/>
+  <xacro:property name="object_thickness" value="${yaml_params['object_thickness']}"/>
+  <xacro:property name="object_inscribed_radius" value="${yaml_params['object_inscribed_radius']}"/>
   <!-- Compute inertial properties for a cylinder, where the reference frame is centered.
        The axis of the cylinder
@@ -330,5 +336,5 @@
       <axis xyz="0 0 1" />
       <!-- Limits are required but currently arbitrary -->
-      <limit lower="${-base_offset}" upper="${vert_limit}" effort="100" velocity="100"/>
+      <limit lower="0" upper="${vert_limit}" effort="100" velocity="100"/>
       <dynamics damping="0.0" friction="0.0"/>
     </joint>
@@ -355,8 +361,12 @@
     <xacro:end_effector tail_id="3" prefix="${prefix}"/>
   </xacro:macro>
+<!--
+  NOTE: PLEASE DO NOT CHANGE THIS SECTION, AS OMNID_PLANNING_ADAPTER_PLUGIN
+  DEPENDS DIRECTLY ON CONFIGURATIONS HERE
+-->
   <xacro:macro name="object_platform">
     <joint name="object_platform/fixed" type="fixed">
       <parent link="world"/>
-      <origin xyz="${object_platform_base_x} ${object_platform_base_y} ${object_platform_base_z-base_offset}"/>
+      <origin xyz="${object_platform_base_x} ${object_platform_base_y} ${object_platform_base_z + object_clearance + object_thickness/2.0}"/>
       <child link="object_platform_base"/>
     </joint>
@@ -386,6 +396,25 @@
     </joint>
     <link name="object_platform_z_link"/>
+    <!--  we are following the ROS yaw-pitch-row convention-->
+    <joint name="object_platform/yaw" type="revolute" >
+      <parent link="object_platform_z_link" />
+      <child link="object_platform_yaw_link" />
+      <origin xyz="0 0 0" rpy="0 0 0" />
+      <axis xyz="0 0 1" rpy="0 0 0"/>
+      <limit lower="${-pi/2.0}" upper="${pi/2.0}" effort="100" velocity="100" />
+      <dynamics damping="0.0" friction="0.0"/>
+    </joint>
+    <link name="object_platform_yaw_link"/>
+    <joint name="object_platform/pitch" type="revolute" >
+      <parent link="object_platform_yaw_link" />
+      <child link="object_platform_pitch_link" />
+      <origin xyz="0 0 0" rpy="0 0 0" />
+      <axis xyz="0 1 0" rpy="0 0 0"/>
+      <limit lower="${-pi/2.0}" upper="${pi/2.0}" effort="100" velocity="100" />
+      <dynamics damping="0.0" friction="0.0"/>
+    </joint>
+    <link name="object_platform_pitch_link"/>
     <joint name="object_platform/roll" type="revolute" >
-      <parent link="object_platform_z_link" />
+      <parent link="object_platform_pitch_link" />
       <child link="object_platform_roll_link" />
       <origin xyz="0 0 0" rpy="0 0 0" />
@@ -395,28 +424,17 @@
     </joint>
     <link name="object_platform_roll_link"/>
-    <joint name="object_platform/pitch" type="revolute" >
-      <parent link="object_platform_roll_link" />
-      <child link="object_platform_pitch_link" />
-      <origin xyz="0 0 0" rpy="0 0 0" />
-      <axis xyz="0 1 0" rpy="0 0 0"/>
-      <limit lower="${-pi/2.0}" upper="${pi/2.0}" effort="100" velocity="100" />
-      <dynamics damping="0.0" friction="0.0"/>
-    </joint>
-    <link name="object_platform_pitch_link"/>
-    <joint name="object_platform/yaw" type="revolute" >
-      <parent link="object_platform_pitch_link" />
-      <child link="object_platform_yaw_link" />
-      <origin xyz="0 0 0" rpy="0 0 0" />
-      <axis xyz="0 0 1" rpy="0 0 0"/>
-      <limit lower="${-pi/2.0}" upper="${pi/2.0}" effort="100" velocity="100" />
-      <dynamics damping="0.0" friction="0.0"/>
-    </joint>
-    <link name="object_platform_yaw_link"/>
     <joint name="object_platform_eef" type="fixed">
-      <parent link="object_platform_yaw_link"/>
+      <parent link="object_platform_roll_link"/>
       <origin xyz="0 0 0"/>
       <child link="object_platform_end_effector"/>
     </joint>
-    <link name="object_platform_end_effector"/>
+<!--    <link name="object_platform_end_effector"/>-->
+<!--    TODO-->
+    <xacro:cylinder_link name="object_platform_end_effector"
+                         M="${M_platform}"
+                         R="${object_inscribed_radius}"
+                         h="${object_thickness}"
+                         axis="z"
+                         mat="dark_pink" />
   </xacro:macro>
 <!--  robot group set up. All arms are internally connected to the world link -->

Commit message: Updated README.md

File: omnid/urdf/delta_robot_group_moveit.urdf.xacro (robot description, xacro)
@@ -83,5 +83,4 @@
   <xacro:property name="yaml_file" value="$(find omnid)/params/params.yaml"/>
   <xacro:property name="yaml_params" value="${load_yaml(yaml_file)}"/>
-  <xacro:property name="object_clearance" value="${yaml_params['object_clearance']}"/>
   <xacro:property name="object_thickness" value="${yaml_params['object_thickness']}"/>
   <xacro:property name="object_inscribed_radius" value="${yaml_params['object_inscribed_radius']}"/>
@@ -368,5 +367,5 @@
     <joint name="object_platform/fixed" type="fixed">
       <parent link="world"/>
-      <origin xyz="${object_platform_base_x} ${object_platform_base_y} ${object_platform_base_z + object_clearance + object_thickness/2.0}"/>
+      <origin xyz="${object_platform_base_x} ${object_platform_base_y} ${object_platform_base_z}"/>
       <child link="object_platform_base"/>
     </joint>

File: omnid/urdf/delta_robot_pybullet.urdf (robot description, URDF)
Before this commit: robot delta-robot-RUU, 20 links, 19 joints
Joints:
- joint lower_leg_attach_joint_2: origin xyz=-0.09 0.155884572681 0 rpy=0 0 2.09439510239 -> xyz=-0.08999999999999996 0.15588457268119896 0 rpy=0 0 2.0943951023931953
- joint lower_leg_attach_joint_3: origin xyz=-0.09 -0.155884572681 0 rpy=0 0 4.18879020479 -> xyz=-0.09000000000000008 -0.1558845726811989 0 rpy=0 0 4.1887902047863905
- joint phi_1: origin xyz=0 -0.09 0 rpy=0 0 1.57079632679 -> xyz=0 -0.09 0 rpy=0 0 1.5707963267948966
- joint phi_2: origin xyz=0 -0.09 0 rpy=0 0 1.57079632679 -> xyz=0 -0.09 0 rpy=0 0 1.5707963267948966
- joint phi_3: origin xyz=0 -0.09 0 rpy=0 0 1.57079632679 -> xyz=0 -0.09 0 rpy=0 0 1.5707963267948966
- joint theta_1: limit lower=-0.785398163397 upper=1.57079632679 effort=100 velocity=100 -> lower=-0.7853981633974483 upper=1.5707963267948966 effort=100 velocity=100
- joint theta_2: limit lower=-0.785398163397 upper=1.57079632679 effort=100 velocity=100 -> lower=-0.7853981633974483 upper=1.5707963267948966 effort=100 velocity=100
- joint theta_3: limit lower=-0.785398163397 upper=1.57079632679 effort=100 velocity=100 -> lower=-0.7853981633974483 upper=1.5707963267948966 effort=100 velocity=100
- joint z: limit lower=-0.046375 upper=0.568 effort=100 velocity=100 -> lower=-0.046375 upper=0.5680000000000001 effort=100 velocity=100

File: omnid/urdf/disk.urdf (robot description, URDF)
Before this commit: robot disk, 1 links, 0 joints
Links:
- link base_link: geometry collision cylinder length=0.01 radius=0.8; visual cylinder length=0.01 radius=0.8

File: omnid/urdf/disk.urdf.xacro (robot description, xacro)
@@ -3,9 +3,11 @@
   <!--  a circular disk object for carrying. The link frame is positioned at the bottom of the link -->
   <!-- Radius of the base of the delta robot -->
-  <xacro:property name="R_disk" value="$(arg R_disk)" />
+  <xacro:property name="yaml_file"    value="$(find omnid)/params/params.yaml" />
+  <xacro:property name="properties"   value="${load_yaml(yaml_file)}" />
+  <xacro:property name="R_disk" value="${properties['object_inscribed_radius']}" />
   <!-- height (i.e. thickness) of the base -->
-  <xacro:property name="h_disk" value="$(arg h_disk)" />
+  <xacro:property name="h_disk" value="${properties['object_thickness']}" />
   <!-- mass of the base -->
-  <xacro:property name="M_disk" value="$(arg M_disk)" />
+  <xacro:property name="M_disk" value="${properties['object_mass']}" />
   <!-- Compute inertial properties for a cylinder, where the reference frame is centered.
        The axis of the cylinder-->
@@ -67,4 +69,5 @@
   </material>
   <!-- define the base of the delta robot-->
+  <link name="world"/>
   <xacro:cylinder_link name="base_link"
                          M="${M_disk}"
